Commit message: working git status!

File: src/enph353_ros_lab/urdf/macros.xacro (robot description, xacro)
@@ -34,5 +34,5 @@
   </macro>
   <macro name="castor_visual"  params="x y z r p yaw radius">
-    <visual name="wheel_visual">
+    <visual name="castor_visual">
       <origin xyz="${x} ${y} ${z}" rpy=" ${r} ${p} ${yaw}"/>
        <geometry>

File: src/enph353_ros_lab/urdf/robot.xacro (robot description, xacro)
@@ -7,7 +7,7 @@
   <xacro:property name="wheel_radius" value="0.04"/>
   <xacro:property name="wheel_width" value="0.03"/>
-  <xacro:property name="wheel_mass" value="0.075"/>
-  <xacro:property name="castor_radius" value="0.025"/>
-  <xacro:property name="castor_mass" value="0.1"/>
+  <xacro:property name="wheel_mass" value="0.15"/>
+  <xacro:property name="castor_radius" value="0.03"/>
+  <xacro:property name="castor_mass" value="0.3"/>
   <xacro:property name="camera_link" value="0.05" /> <!-- Size of square 'camera' box -->
   <!-- <xacro:include filename="$(find enph353_ros_lab)/urdf/robot.gazebo" /> -->
@@ -40,33 +40,51 @@
     </visual>
   </link>
-  <link name="castor">
+  <!-- <link name="castor">
     <xacro:sphere_inertial name="castor" m="${castor_mass}" r="${castor_radius}" />
     <xacro:castor_collision radius="${castor_radius}" x="0" y="0" z="0" r="0" p="0" yaw="0"/>
     <xacro:castor_visual x="0" y="0" z="0" r="0" p="0" yaw="0" radius="${castor_radius}" />
+  </link> -->
+  <link name="topleftwheel">
+    <xacro:cylinder_inertial name="topleftwheel" m="${wheel_mass}" r="${wheel_radius}" h="${wheel_width}"/>
+    <xacro:wheel_collision radius="${wheel_radius}" width="${wheel_width}" x="0" y="0" z="0" r="1.570595" p="0" yaw="0"/>
+    <xacro:wheel_visual x="0" y="0" z="0" r="1.570595" p="0" yaw="0" radius="${wheel_radius}" width="${wheel_width}"/>
+  </link>
+  <link name="toprightwheel">
+    <xacro:cylinder_inertial name="toprightwheel" m="${wheel_mass}" r="${wheel_radius}" h="${wheel_width}"/>
+    <xacro:wheel_collision radius="${wheel_radius}" width="${wheel_width}" x="0" y="0" z="0" r="1.570595" p="0" yaw="0"/>
+    <xacro:wheel_visual x="0" y="0" z="0" r="1.570595" p="0" yaw="0" radius="${wheel_radius}" width="${wheel_width}"/>
   </link>
   <link name="bottomleftwheel">
-    <xacro:cylinder_inertial name="topleftwheel" m="${wheel_mass}" r="${wheel_radius}" h="${wheel_width}"/>
-    <xacro:wheel_collision radius="${wheel_radius}" width="${wheel_width}" x="0" y="0" z="0" r="1.57" p="0" yaw="0"/>
-    <xacro:wheel_visual x="0" y="0" z="0" r="1.57" p="0" yaw="0" radius="${wheel_radius}" width="${wheel_width}"/>
+    <xacro:cylinder_inertial name="bottomleftwheel" m="${wheel_mass}" r="${wheel_radius}" h="${wheel_width}"/>
+    <xacro:wheel_collision radius="${wheel_radius}" width="${wheel_width}" x="0" y="0" z="0" r="1.570595" p="0" yaw="0"/>
+    <xacro:wheel_visual x="0" y="0" z="0" r="1.570595" p="0" yaw="0" radius="${wheel_radius}" width="${wheel_width}"/>
   </link>
   <link name="bottomrightwheel">
-    <xacro:cylinder_inertial name="topleftwheel" m="${wheel_mass}" r="${wheel_radius}" h="${wheel_width}"/>
-    <xacro:wheel_collision radius="${wheel_radius}" width="${wheel_width}" x="0" y="0" z="0" r="-1.57" p="0" yaw="0"/>
-    <xacro:wheel_visual x="0" y="0" z="0" r="-1.57" p="0" yaw="0" radius="${wheel_radius}" width="${wheel_width}"/>
+    <xacro:cylinder_inertial name="bottomrightwheel" m="${wheel_mass}" r="${wheel_radius}" h="${wheel_width}"/>
+    <xacro:wheel_collision radius="${wheel_radius}" width="${wheel_width}" x="0" y="0" z="0" r="1.570595" p="0" yaw="0"/>
+    <xacro:wheel_visual x="0" y="0" z="0" r="1.570595" p="0" yaw="0" radius="${wheel_radius}" width="${wheel_width}"/>
   </link>
- <joint name="castorjoint" type ="continuous">
-    <xacro:castor_joint x="0.075" y="0" z="-0.02" r="0" p="0" yaw="0" parentlink="chassis" childlink="castor"/>
+ <!-- <joint name="castorjoint" type ="continuous">
+    <xacro:castor_joint x="0.07" y="0" z="-0.02" r="0" p="0" yaw="0" parentlink="chassis" childlink="castor"/>
+  </joint>  -->
+  <joint name="topleftwheeljoint" type ="continuous">
+    <xacro:wheel_joint x="0.075" y="0.09" z="-0.01" r="0" p="0" yaw="0" parentlink="chassis" childlink="topleftwheel"/>
+    <axis xyz="0 1 0"/>
+  </joint>
+  <joint name="toprightwheeljoint" type ="continuous">
+    <xacro:wheel_joint x="0.075" y="-0.09" z="-0.01" r="0" p="0" yaw="0" parentlink="chassis" childlink="toprightwheel"/>
+    <axis xyz="0 1 0"/>
   </joint>
   <joint name="bottomleftwheeljoint" type ="continuous">
-    <xacro:wheel_joint x="-0.075" y="0.10" z="-0.03" r="0" p="0" yaw="0" parentlink="chassis" childlink="bottomleftwheel"/>
+    <xacro:wheel_joint x="-0.075" y="0.09" z="-0.01" r="0" p="0" yaw="0" parentlink="chassis" childlink="bottomleftwheel"/>
     <axis xyz="0 1 0"/>
   </joint>
   <joint name="bottomrightwheeljoint" type ="continuous">
-    <xacro:wheel_joint x="-0.075" y="-0.10" z="-0.03" r="0" p="0" yaw="0" parentlink="chassis" childlink="bottomrightwheel"/>
+    <xacro:wheel_joint x="-0.075" y="-0.09" z="-0.01" r="0" p="0" yaw="0" parentlink="chassis" childlink="bottomrightwheel"/>
     <axis xyz="0 1 0"/>
   </joint>
   <joint name="camera_joint" type="fixed">
     <axis xyz="0 1 0" />
-    <origin xyz="${camera_link} 0 ${0.05 - 0.01*2}" rpy="0 0 0"/>
+    <origin xyz="${camera_link} 0 0.05" rpy="0 0 0"/>
     <parent link="chassis"/>
     <child link="camera_link"/>
@@ -93,5 +111,21 @@
     </inertial>
   </link>
-<gazebo>
+  <gazebo>
+        <plugin name="skid_steer_drive_controller" filename="libgazebo_ros_skid_steer_drive.so">
+	     <updateRate>20.0</updateRate>
+	     <robotNamespace>/</robotNamespace>
+	     <leftFrontJoint>topleftwheeljoint</leftFrontJoint>
+	     <rightFrontJoint>toprightwheeljoint</rightFrontJoint>
+	     <leftRearJoint>bottomleftwheeljoint</leftRearJoint>
+	     <rightRearJoint>bottomrightwheeljoint</rightRearJoint>
+	     <wheelSeparation>0.18</wheelSeparation>
+	     <wheelDiameter>0.08</wheelDiameter>
+	     <robotBaseFrame>base_link</robotBaseFrame>
+	     <torque>20</torque>
+	     <topicName>cmd_vel</topicName>
+	     <broadcastTF>false</broadcastTF>
+        </plugin>
+  </gazebo>
+<!-- <gazebo>
   <plugin name="differential_drive_controller" filename="libgazebo_ros_diff_drive.so">
     <alwaysOn>true</alwaysOn>
@@ -99,6 +133,6 @@
     <leftJoint>base_link_right_wheel_joint</leftJoint>
     <rightJoint>base_link_left_wheel_joint</rightJoint>
-    <wheelSeparation>0.5380</wheelSeparation>
-    <wheelDiameter>0.2410</wheelDiameter>
+    <wheelSeparation>0.160</wheelSeparation>
+    <wheelDiameter>0.08</wheelDiameter>
     <torque>20</torque>
     <commandTopic>cmd_vel</commandTopic>
@@ -107,5 +141,5 @@
     <robotBaseFrame>base_footprint</robotBaseFrame>
   </plugin>
-</gazebo>
+</gazebo>  -->
 <!-- camera -->
 <gazebo reference="camera_link">
